File: KiCad/Shaviry.kicad_sch (KiCad schematic)
At the start: 27 parts, among them J1 AMIGA_DB23_RGB_ENTRADA_HEMBRA, J2 VGA_SALIDA_HEMBRA, J3 VGA_ENTRADA_HEMBRA, J4 Conn_02x03_Top_Bottom, J5 Conn_01x03_Pin, U1 74HCT14, U3 THS7374, U5 PC817

Commit message: Add files via upload
Connections:
- net at R5.1: now also U3.12 (CH3_OUT); no longer U3.13 (CH2_OUT)
- net at R6.1: now also U3.11 (CH4_OUT); no longer U3.12 (CH3_OUT)
- net at J1.3 (RED), R1.2: now also U3.2 (CH2_IN); no longer U3.1 (CH1_IN)
- net at J1.4 (GREEN), R2.2: now also U3.3 (CH3_IN); no longer U3.2 (CH2_IN)
- net at J1.5 (BLUE), R3.2: now also U3.4 (CH4_IN); no longer U3.3 (CH3_IN)
- net at R4.1: now also U3.13 (CH2_OUT); no longer U3.14 (CH1_OUT)
Other:
- moved on the sheet: R1, R2, R3
